File: Hardware/Electronics/Control Board.brd (EAGLE design)
At the start: 65 x 55 mm, 13 parts, among them J1 22-27-2041-04, J2 22-27-2021-02, Q2 BUZ11BV, U1 V_REG_317SMD, X1 22-23-2031

Commit message: Intermediate commit - needs improvement
Parts:
- removed C1, C2: (no value), resistor:E2,5-7
- moved U1 40.8 mm to (29.6, 7.92), turned to 180 degrees
- moved PAD 22.1 mm to (41.1, 41.9)
- moved J2 9.69 mm to (48.9, 38.1)
Connections:
- new net N$10: U$1.D4, U$2.RST
- net +12V: no longer C1.+
- net +3V3: now also U$2.CH_PD; no longer C2.+
- net GND: no longer C1.-, C2.-
- net N$2: now also U$1.D3; no longer U$1.RXO
- net N$3: now also U$1.D2; no longer U$1.TXI
- net N$4: now also U$1.D9; no longer U$1.D3
- net N$5: now also U$1.D10; no longer U$1.D4
- net N$6: now also U$1.D11; no longer U$1.D5
- net N$7: now also U$1.D12; no longer U$1.D6
- net UV-SWITCH: no longer U$1.A7
Routing:
- net +12V: track 70.8 -> 121.3 mm, vias 0 -> 2
- net GND: track 163.7 -> 137.9 mm
- net +3V3: track 47.7 -> 27.9 mm, vias 2 -> 0
- net N$2: track 8.89 -> 26.7 mm
- net N$7: track 21.6 -> 5.60 mm
- net N$6: track 21.6 -> 5.60 mm
- net N$5: track 21.6 -> 5.60 mm
- net N$4: track 21.6 -> 5.60 mm
- net N$3: track 31.7 -> 21.6 mm
- net UV-SWITCH: track 18.4 -> 15.9 mm

Commit message: Electronics - Working version
Parts:
- moved U1 3.17 mm to (29.6, 4.74), flipped to the top
Connections:
- net UV-SWITCH: now also U$1.A5
Routing:
- net N$10: track 0.00 -> 39.4 mm
- net +12V: track 121.3 -> 126.8 mm
- net GND: track 137.9 -> 142.5 mm, vias 0 -> 1
- net +3V3: track 27.9 -> 30.5 mm
- net UV-SWITCH: track 15.9 -> 17.1 mm
Changed lines of the file:
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@@
 <hole x="62" y="3" drill="1.4"/>
 <hole x="62" y="52" drill="1.4"/>
-<text x="33" y="31" size="1.778" layer="16" rot="MR270">UV-Led Control Board</text>
+<text x="30.46" y="41.16" size="1.778" layer="16" rot="MR270">UV-Led Control Board</text>
 </plain>
 <attributes>
@@
 <element name="U$1" library="MimaZ" package="ARDUINO_NANO_V3" value="ARDUINO_NANO_V3" x="35.56" y="8.89" rot="R180"/>
 <element name="U$2" library="MimaZ" package="ESP8266" value="ESP8266" x="41.91" y="30.48" rot="R270"/>
-<element name="U1" library="SparkFun-PowerIC" package="SOT223" value="V_REG_317SMD" x="29.645" y="7.915" rot="MR180"/>
+<element name="U1" library="SparkFun-PowerIC" package="SOT223" value="V_REG_317SMD" x="29.645" y="4.74" rot="R180"/>
 <element name="J1" library="con-molex" package="6410-04" value="22-27-2041-04" x="10.795" y="41.275" rot="R270">
 <attribute name="OC_NEWARK" value="unknown" x="10.795" y="41.275" size="1.778" layer="27" rot="R270" display="off"/>
@@
 <wire x1="8.255" y1="8.255" x2="8.255" y2="11.43" width="1.27" layer="16"/>
 <wire x1="22.86" y1="11.43" x2="25.4" y2="11.43" width="1.27" layer="16"/>
-<wire x1="25.4" y1="11.0138" x2="25.4" y2="5.08" width="1.27" layer="16"/>
-<wire x1="25.4" y1="5.08" x2="8.255" y2="5.08" width="1.27" layer="16"/>
-<wire x1="8.255" y1="5.08" x2="8.255" y2="8.255" width="1.27" layer="16"/>
 <wire x1="10.795" y1="45.085" x2="17.145" y2="45.085" width="1.27" layer="16"/>
 <wire x1="17.145" y1="45.085" x2="17.145" y2="46.99" width="1.27" layer="16"/>
@@
 <wire x1="41.15" y1="47.004" x2="25.4" y2="47.004" width="1.27" layer="16"/>
 <wire x1="25.4" y1="47.004" x2="25.4" y2="46.99" width="1.27" layer="16"/>
+<wire x1="25.4" y1="11.0138" x2="25.4" y2="11.43" width="1.27" layer="16"/>
+<via x="25.4" y="11.0138" extent="1-16" drill="0.6" shape="square"/>
+<wire x1="31.9564" y1="7.8388" x2="31.75" y2="7.8388" width="1.27" layer="1"/>
+<wire x1="31.75" y1="7.8388" x2="31.75" y2="12.065" width="1.27" layer="1"/>
+<wire x1="31.75" y1="12.065" x2="25.4" y2="12.065" width="1.27" layer="1"/>
+<wire x1="25.4" y1="12.065" x2="25.4" y2="11.0138" width="1.27" layer="1"/>
 <wire x1="25.4" y1="46.99" x2="30.734" y2="43.053" width="0" layer="19" extent="1-16"/>
-<wire x1="35.56" y1="16.51" x2="27.3336" y2="11.0138" width="0" layer="19" extent="16-16"/>
-<wire x1="27.3336" y1="11.0138" x2="25.4" y2="11.0138" width="1.27" layer="16"/>
-<wire x1="25.4" y1="11.0138" x2="25.4" y2="11.43" width="1.27" layer="16"/>
+<wire x1="35.56" y1="16.51" x2="31.75" y2="12.065" width="0" layer="19" extent="1-1"/>
+<wire x1="8.255" y1="11.43" x2="8.255" y2="14.605" width="1.27" layer="1"/>
+<wire x1="8.255" y1="14.605" x2="19.685" y2="14.605" width="1.27" layer="1"/>
+<wire x1="19.685" y1="14.605" x2="19.685" y2="11.43" width="1.27" layer="1"/>
+<wire x1="19.685" y1="11.43" x2="22.86" y2="11.43" width="1.27" layer="1"/>
 </signal>
 <signal name="+12V">
@@
 <wire x1="45.72" y1="39.37" x2="48.895" y2="39.37" width="1.27" layer="16"/>
 <wire x1="15.875" y1="48.895" x2="28.194" y2="43.053" width="0" layer="19" extent="1-16"/>
-<wire x1="31.9564" y1="11.0138" x2="22.86" y2="8.89" width="0" layer="19" extent="16-16"/>
+<wire x1="27.3336" y1="7.8388" x2="22.86" y2="7.8388" width="1.27" layer="1"/>
+<wire x1="22.86" y1="7.8388" x2="22.86" y2="8.89" width="1.27" layer="1"/>
 </signal>
 <signal name="UV-SWITCH">
@@
 <wire x1="10.795" y1="22.225" x2="13.335" y2="22.225" width="1.27" layer="16"/>
 <wire x1="13.335" y1="22.225" x2="13.335" y2="19.05" width="1.27" layer="16"/>
-<wire x1="20.32" y1="19.05" x2="20.32" y2="22.225" width="1.27" layer="16"/>
 <via x="20.32" y="22.225" extent="1-16" drill="0.6" shape="square"/>
 <wire x1="20.32" y1="22.225" x2="13.335" y2="22.225" width="1.27" layer="1"/>
 <via x="13.335" y="22.225" extent="1-16" drill="0.6" shape="square"/>
+<contactref element="U$1" pad="A5"/>
+<wire x1="20.32" y1="22.225" x2="20.32" y2="24.13" width="1.27" layer="16"/>
+<wire x1="20.32" y1="24.13" x2="22.86" y2="24.13" width="1.27" layer="16"/>
 </signal>
 <signal name="N$3">
@@
 <wire x1="49.53" y1="5.08" x2="44.45" y2="5.08" width="1.27" layer="16"/>
 <contactref element="U$2" pad="CH_PD"/>
-<wire x1="44.45" y1="5.08" x2="29.21" y2="5.08" width="1.27" layer="16"/>
 <wire x1="44.45" y1="8.89" x2="44.45" y2="5.08" width="1.27" layer="16"/>
-<wire x1="29.21" y1="5.08" x2="29.645" y2="11.0138" width="0" layer="19" extent="16-16"/>
+<wire x1="29.21" y1="5.08" x2="29.645" y2="7.8388" width="0" layer="19" extent="16-16"/>
+<wire x1="44.45" y1="5.08" x2="29.845" y2="5.08" width="1.27" layer="16"/>
+<wire x1="29.845" y1="5.08" x2="29.845" y2="1.905" width="1.27" layer="16"/>
+<wire x1="29.845" y1="1.905" x2="29.645" y2="7.8388" width="0" layer="19" extent="1-16"/>
 </signal>
 <signal name="N$2">
@@
 <contactref element="U$2" pad="RST"/>
 <contactref element="U$1" pad="D4"/>
-<wire x1="46.99" y1="8.89" x2="35.56" y2="24.13" width="0" layer="19" extent="1-1"/>
+<wire x1="46.99" y1="8.89" x2="46.99" y2="6.985" width="1.27" layer="1"/>
+<wire x1="46.99" y1="6.985" x2="51.435" y2="6.985" width="1.27" layer="1"/>
+<wire x1="51.435" y1="6.985" x2="51.435" y2="24.13" width="1.27" layer="1"/>
+<wire x1="51.435" y1="24.13" x2="35.56" y2="24.13" width="1.27" layer="1"/>
 </signal>
 </signals>
