File: Hardware/Electronics/Control Board.sch (EAGLE design)
At the start: 13 parts, among them J1 22-27-2041-04, J2 22-27-2021-02, Q2 BUZ11BV, U1 V_REG_317SMD, X1 22-23-2031

Commit message: Intermediate commit - needs improvement
Parts:
- removed C1, C2: (no value), resistor:CPOL-EUE2.5-7
Connections:
- new net N$10: U$1.D4, U$2.RST
- net +12V: no longer C1.+
- net +3V3: now also U$2.CH_PD; no longer C2.+
- net GND: no longer C1.-, C2.-
- net N$2: now also U$1.D3; no longer U$1.RXO
- net N$3: now also U$1.D2; no longer U$1.TXI
- net N$4: now also U$1.D9; no longer U$1.D3
- net N$5: now also U$1.D10; no longer U$1.D4
- net N$6: now also U$1.D11; no longer U$1.D5
- net N$7: now also U$1.D12; no longer U$1.D6
- net UV-SWITCH: no longer U$1.A7
Other:
- note added: "1"
- note removed: "0"
- moved on the sheet: PAD-1, PAD-2, PAD-3, PAD-4, PAD-5
Changed lines of the file:
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@@
 <part name="U$2" library="MimaZ" deviceset="ESP8266" device=""/>
 <part name="U1" library="SparkFun-PowerIC" deviceset="V_REG_317" device="SMD"/>
-<part name="C1" library="resistor" deviceset="CPOL-EU" device="E2.5-7"/>
-<part name="C2" library="resistor" deviceset="CPOL-EU" device="E2.5-7"/>
 <part name="P+3" library="supply1" deviceset="+12V" device=""/>
 <part name="GND4" library="supply1" deviceset="GND" device=""/>
@@
 <part name="P+6" library="supply1" deviceset="+12V" device=""/>
 <part name="GND8" library="supply1" deviceset="GND" device=""/>
+<part name="+3V3" library="supply1" deviceset="+3V3" device=""/>
 </parts>
 <sheets>
@@
 <text x="135.89" y="172.72" size="5.08" layer="94">LCD Screen</text>
 <text x="163.83" y="27.94" size="2.54" layer="94" font="vector">Author: Angel Hernandez</text>
-<text x="256.54" y="7.62" size="2.54" layer="94" font="vector">0</text>
 <text x="17.78" y="166.37" size="2.54" layer="94">12V Input</text>
 <text x="78.74" y="166.37" size="2.54" layer="94">3.3V Regulator</text>
@@
 <wire x1="162.56" y1="119.38" x2="162.56" y2="132.08" width="0.1524" layer="94"/>
 <wire x1="162.56" y1="132.08" x2="165.1" y2="132.08" width="0.1524" layer="94"/>
+<text x="256.54" y="7.62" size="2.54" layer="94">1</text>
 </plain>
 <instances>
@@
 <instance part="U$2" gate="G$1" x="64.77" y="63.5" rot="R180"/>
 <instance part="U1" gate="G$1" x="90.17" y="153.67"/>
-<instance part="C1" gate="G$1" x="73.66" y="149.86"/>
-<instance part="C2" gate="G$1" x="107.95" y="149.86"/>
 <instance part="P+3" gate="1" x="73.66" y="161.29"/>
 <instance part="GND4" gate="1" x="90.17" y="138.43"/>
@@
 <instance part="R6" gate="G$1" x="217.17" y="156.21" rot="R270"/>
 <instance part="Q2" gate="1" x="229.87" y="152.4"/>
-<instance part="PAD" gate="-1" x="64.77" y="58.42" smashed="yes" rot="MR0">
-<attribute name="NAME" x="62.23" y="57.658" size="1.524" layer="95" rot="MR0"/>
-<attribute name="VALUE" x="65.532" y="59.817" size="1.778" layer="96" rot="MR0"/>
+<instance part="PAD" gate="-1" x="81.28" y="43.18" smashed="yes" rot="MR0">
+<attribute name="NAME" x="78.74" y="42.418" size="1.524" layer="95" rot="MR0"/>
+<attribute name="VALUE" x="82.042" y="44.577" size="1.778" layer="96" rot="MR0"/>
 </instance>
-<instance part="PAD" gate="-2" x="64.77" y="55.88" rot="MR0"/>
-<instance part="PAD" gate="-3" x="64.77" y="53.34" rot="MR0"/>
-<instance part="PAD" gate="-4" x="64.77" y="50.8" rot="MR0"/>
-<instance part="PAD" gate="-5" x="64.77" y="48.26" rot="MR0"/>
-<instance part="GND7" gate="1" x="69.85" y="43.18"/>
+<instance part="PAD" gate="-2" x="81.28" y="40.64" rot="MR0"/>
+<instance part="PAD" gate="-3" x="81.28" y="38.1" rot="MR0"/>
+<instance part="PAD" gate="-4" x="81.28" y="35.56" rot="MR0"/>
+<instance part="PAD" gate="-5" x="81.28" y="33.02" rot="MR0"/>
+<instance part="GND7" gate="1" x="86.36" y="27.94"/>
 <instance part="J2" gate="-1" x="26.67" y="152.4" rot="MR0"/>
 <instance part="J2" gate="-2" x="26.67" y="147.32" rot="MR0"/>
 <instance part="P+6" gate="1" x="33.02" y="160.02"/>
 <instance part="GND8" gate="1" x="33.02" y="140.97"/>
+<instance part="+3V3" gate="G$1" x="76.2" y="109.22"/>
 </instances>
 <busses>
@@
 </segment>
 <segment>
-<pinref part="C1" gate="G$1" pin="-"/>
-<wire x1="73.66" y1="144.78" x2="90.17" y2="144.78" width="0.1524" layer="91"/>
 <pinref part="U1" gate="G$1" pin="ADJ"/>
-<wire x1="90.17" y1="144.78" x2="90.17" y2="146.05" width="0.1524" layer="91"/>
 <pinref part="GND4" gate="1" pin="GND"/>
-<wire x1="90.17" y1="140.97" x2="90.17" y2="144.78" width="0.1524" layer="91"/>
-<junction x="90.17" y="144.78"/>
-<pinref part="C2" gate="G$1" pin="-"/>
-<wire x1="107.95" y1="144.78" x2="90.17" y2="144.78" width="0.1524" layer="91"/>
+<wire x1="90.17" y1="140.97" x2="90.17" y2="146.05" width="0.1524" layer="91"/>
 </segment>
 <segment>
@@
 <pinref part="PAD" gate="-5" pin="S"/>
 <pinref part="GND7" gate="1" pin="GND"/>
-<wire x1="67.31" y1="48.26" x2="69.85" y2="48.26" width="0.1524" layer="91"/>
-<wire x1="69.85" y1="48.26" x2="69.85" y2="45.72" width="0.1524" layer="91"/>
+<wire x1="83.82" y1="33.02" x2="86.36" y2="33.02" width="0.1524" layer="91"/>
+<wire x1="86.36" y1="33.02" x2="86.36" y2="30.48" width="0.1524" layer="91"/>
 </segment>
 <segment>
@@
 <segment>
 <pinref part="P+3" gate="1" pin="+12V"/>
-<pinref part="C1" gate="G$1" pin="+"/>
 <wire x1="73.66" y1="158.75" x2="73.66" y2="153.67" width="0.1524" layer="91"/>
 <pinref part="U1" gate="G$1" pin="IN"/>
-<wire x1="73.66" y1="153.67" x2="73.66" y2="152.4" width="0.1524" layer="91"/>
 <wire x1="82.55" y1="153.67" x2="73.66" y2="153.67" width="0.1524" layer="91"/>
-<junction x="73.66" y="153.67"/>
 </segment>
 <segment>
@@
 <net name="UV-SWITCH" class="0">
 <segment>
-<label x="138.43" y="49.53" size="1.778" layer="95"/>
-<wire x1="134.62" y1="48.26" x2="152.4" y2="48.26" width="0.1524" layer="91"/>
-<pinref part="U$1" gate="G$1" pin="A7"/>
+<label x="138.43" y="54.61" size="1.778" layer="95"/>
+<wire x1="154.94" y1="53.34" x2="134.62" y2="53.34" width="0.1524" layer="91"/>
 </segment>
 <segment>
@@
 <pinref part="U$2" gate="G$1" pin="RX"/>
 <wire x1="73.66" y1="81.28" x2="69.85" y2="81.28" width="0.1524" layer="91"/>
-<wire x1="73.66" y1="68.58" x2="73.66" y2="81.28" width="0.1524" layer="91"/>
-<pinref part="U$1" gate="G$1" pin="TXI"/>
-<wire x1="73.66" y1="68.58" x2="93.98" y2="68.58" width="0.1524" layer="91"/>
+<wire x1="73.66" y1="60.96" x2="73.66" y2="81.28" width="0.1524" layer="91"/>
+<pinref part="U$1" gate="G$1" pin="D2"/>
+<wire x1="73.66" y1="60.96" x2="93.98" y2="60.96" width="0.1524" layer="91"/>
 </segment>
 </net>
@@
 <segment>
 <pinref part="U1" gate="G$1" pin="OUT"/>
-<pinref part="C2" gate="G$1" pin="+"/>
 <wire x1="97.79" y1="153.67" x2="107.95" y2="153.67" width="0.1524" layer="91"/>
-<wire x1="107.95" y1="153.67" x2="107.95" y2="152.4" width="0.1524" layer="91"/>
 <pinref part="+3V1" gate="G$1" pin="+3V3"/>
 <wire x1="107.95" y1="153.67" x2="107.95" y2="160.02" width="0.1524" layer="91"/>
-<junction x="107.95" y="153.67"/>
 </segment>
 <segment>
@@
 <wire x1="35.56" y1="63.5" x2="35.56" y2="69.85" width="0.1524" layer="91"/>
 </segment>
+<segment>
+<pinref part="U$2" gate="G$1" pin="CH_PD"/>
+<pinref part="+3V3" gate="G$1" pin="+3V3"/>
+<wire x1="69.85" y1="101.6" x2="76.2" y2="101.6" width="0.1524" layer="91"/>
+<wire x1="76.2" y1="101.6" x2="76.2" y2="106.68" width="0.1524" layer="91"/>
+</segment>
 </net>
 <net name="N$2" class="0">
 <segment>
 <pinref part="U$2" gate="G$1" pin="TX"/>
-<wire x1="69.85" y1="66.04" x2="69.85" y2="76.2" width="0.1524" layer="91"/>
-<pinref part="U$1" gate="G$1" pin="RXO"/>
-<wire x1="93.98" y1="66.04" x2="69.85" y2="66.04" width="0.1524" layer="91"/>
+<wire x1="69.85" y1="58.42" x2="69.85" y2="76.2" width="0.1524" layer="91"/>
+<pinref part="U$1" gate="G$1" pin="D3"/>
+<wire x1="93.98" y1="58.42" x2="69.85" y2="58.42" width="0.1524" layer="91"/>
 </segment>
 </net>
@@
 </segment>
 </net>
+<net name="N$4" class="0">
+<segment>
+<pinref part="U$1" gate="G$1" pin="D9"/>
+<wire x1="93.98" y1="43.18" x2="83.82" y2="43.18" width="0.1524" layer="91"/>
+<pinref part="PAD" gate="-1" pin="S"/>
+</segment>
+</net>
 <net name="N$5" class="0">
 <segment>
+<pinref part="PAD" gate="-2" pin="S"/>
+<pinref part="U$1" gate="G$1" pin="D10"/>
+<wire x1="83.82" y1="40.64" x2="93.98" y2="40.64" width="0.1524" layer="91"/>
+</segment>
+</net>
+<net name="N$6" class="0">
+<segment>
+<pinref part="U$1" gate="G$1" pin="D11"/>
+<pinref part="PAD" gate="-3" pin="S"/>
+<wire x1="93.98" y1="38.1" x2="83.82" y2="38.1" width="0.1524" layer="91"/>
+</segment>
+</net>
+<net name="N$7" class="0">
+<segment>
+<pinref part="PAD" gate="-4" pin="S"/>
+<pinref part="U$1" gate="G$1" pin="D12"/>
+<wire x1="83.82" y1="35.56" x2="93.98" y2="35.56" width="0.1524" layer="91"/>
+</segment>
+</net>
+<net name="N$10" class="0">
+<segment>
+<pinref part="U$2" gate="G$1" pin="RST"/>
+<wire x1="69.85" y1="96.52" x2="77.47" y2="96.52" width="0.1524" layer="91"/>
+<wire x1="77.47" y1="96.52" x2="77.47" y2="55.88" width="0.1524" layer="91"/>
 <pinref part="U$1" gate="G$1" pin="D4"/>
-<wire x1="93.98" y1="55.88" x2="67.31" y2="55.88" width="0.1524" layer="91"/>
-<pinref part="PAD" gate="-2" pin="S"/>
-</segment>
-</net>
-<net name="N$6" class="0">
-<segment>
-<pinref part="U$1" gate="G$1" pin="D5"/>
-<wire x1="67.31" y1="53.34" x2="93.98" y2="53.34" width="0.1524" layer="91"/>
-<pinref part="PAD" gate="-3" pin="S"/>
-</segment>
-</net>
-<net name="N$7" class="0">
-<segment>
-<pinref part="U$1" gate="G$1" pin="D6"/>
-<wire x1="93.98" y1="50.8" x2="67.31" y2="50.8" width="0.1524" layer="91"/>
-<pinref part="PAD" gate="-4" pin="S"/>
-</segment>
-</net>
-<net name="N$4" class="0">
-<segment>
-<pinref part="U$1" gate="G$1" pin="D3"/>
-<pinref part="PAD" gate="-1" pin="S"/>
-<wire x1="93.98" y1="58.42" x2="67.31" y2="58.42" width="0.1524" layer="91"/>
-</segment>
-</net>
+<wire x1="77.47" y1="55.88" x2="93.98" y2="55.88" width="0.1524" layer="91"/>
+</segment>
+</net>

Commit message: Electronics - Working version
Connections:
- net UV-SWITCH: now also U$1.A5
Changed lines of the file:
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@@
 <setting verticaltext="up"/>
 </settings>
-<grid distance="0.05" unitdist="inch" unit="inch" style="lines" multiple="1" display="no" altdistance="0.01" altunitdist="inch" altunit="inch"/>
+<grid distance="0.1" unitdist="inch" unit="inch" style="lines" multiple="1" display="no" altdistance="0.01" altunitdist="inch" altunit="inch"/>
 <layers>
 <layer number="1" name="Top" color="4" fill="1" visible="no" active="no"/>
@@
 <segment>
 <label x="138.43" y="54.61" size="1.778" layer="95"/>
-<wire x1="154.94" y1="53.34" x2="134.62" y2="53.34" width="0.1524" layer="91"/>
-</segment>
-<segment>
+<wire x1="157.48" y1="53.34" x2="134.62" y2="53.34" width="0.1524" layer="91"/>
+<pinref part="U$1" gate="G$1" pin="A5"/>
+</segment>
+<segment>
